File: _autosave-ultrasonic.sch (KiCad schematic (older format))
At the start: 18 parts, among them J1 10118192-0001LF, J2 Conn_01x03_Male, J3 Conn_01x03_Male, J4 Conn_01x03_Male, U1 CP2102N-A01-GQFN24, U2 ATMEGA328P-AN, U3 LM1117-ADJ

Commit message: Revision 1
Parts:
- J2, J3, J4: footprint Connector_Molex:Molex_Nano-Fit_105309-xx03_1x03_P2.50mm_Vertical -> Connector_Molex:Molex_SL_171971-0003_1x03_P2.54mm_Vertical
- J5: renamed from J?; footprint (none) -> Connector_Molex:Molex_SL_171971-0002_1x02_P2.54mm_Vertical
Changed lines of the file:
@@
 F 0 "J2" H 3408 4681 50  0000 C CNN
 F 1 "Conn_01x03_Male" H 3408 4590 50  0000 C CNN
-F 2 "Connector_Molex:Molex_Nano-Fit_105309-xx03_1x03_P2.50mm_Vertical" H 3300 4400 50  0001 C CNN
+F 2 "Connector_Molex:Molex_SL_171971-0003_1x03_P2.54mm_Vertical" H 3300 4400 50  0001 C CNN
 F 3 "~" H 3300 4400 50  0001 C CNN
 	1    3300 4400
@@
 F 0 "J3" H 3408 5231 50  0000 C CNN
 F 1 "Conn_01x03_Male" H 3408 5140 50  0000 C CNN
-F 2 "Connector_Molex:Molex_Nano-Fit_105309-xx03_1x03_P2.50mm_Vertical" H 3300 4950 50  0001 C CNN
+F 2 "Connector_Molex:Molex_SL_171971-0003_1x03_P2.54mm_Vertical" H 3300 4950 50  0001 C CNN
 F 3 "~" H 3300 4950 50  0001 C CNN
 	1    3300 4950
@@
 F 0 "J4" H 3408 5781 50  0000 C CNN
 F 1 "Conn_01x03_Male" H 3408 5690 50  0000 C CNN
-F 2 "Connector_Molex:Molex_Nano-Fit_105309-xx03_1x03_P2.50mm_Vertical" H 3300 5500 50  0001 C CNN
+F 2 "Connector_Molex:Molex_SL_171971-0003_1x03_P2.54mm_Vertical" H 3300 5500 50  0001 C CNN
 F 3 "~" H 3300 5500 50  0001 C CNN
 	1    3300 5500
@@
 NoConn ~ 5150 4150
 $Comp
-L Connector:Conn_01x02_Male J?
+L Connector:Conn_01x02_Male J5
 U 1 1 5E44608D
 P 2000 4800
-F 0 "J?" H 2108 4981 50  0000 C CNN
+F 0 "J5" H 2108 4981 50  0000 C CNN
 F 1 "Conn_01x02_Male" H 2108 4890 50  0000 C CNN
-F 2 "" H 2000 4800 50  0001 C CNN
+F 2 "Connector_Molex:Molex_SL_171971-0002_1x02_P2.54mm_Vertical" H 2000 4800 50  0001 C CNN
 F 3 "~" H 2000 4800 50  0001 C CNN
 	1    2000 4800
@@
 $EndComp
 $Comp
-L power:+12V #PWR?
+L power:+12V #PWR0120
 U 1 1 5E45295A
 P 2400 4800
-F 0 "#PWR?" H 2400 4650 50  0001 C CNN
+F 0 "#PWR0120" H 2400 4650 50  0001 C CNN
 F 1 "+12V" V 2415 4928 50  0000 L CNN
 F 2 "" H 2400 4800 50  0001 C CNN
@@
 $EndComp
 $Comp
-L power:GND #PWR?
+L power:GND #PWR0121
 U 1 1 5E45301C
 P 2400 4900
-F 0 "#PWR?" H 2400 4650 50  0001 C CNN
+F 0 "#PWR0121" H 2400 4650 50  0001 C CNN
 F 1 "GND" H 2405 4727 50  0000 C CNN
 F 2 "" H 2400 4900 50  0001 C CNN
